Commit message: Declare the passive front wheels to ros2_control
The front road wheels free-wheel, so nothing claimed them and they were
left out of the ros2_control block. That was not cosmetic:
joint_state_broadcaster only publishes joints it knows about, so
robot_state_publisher could not compute front_{left,right}_wheel_link and
those two frames were missing from TF entirely. RViz reported it on the
RobotModel display, which is how it surfaced.

Fixed by listing them with state_interface only, no command_interface.
Verified: /joint_states now carries 6 joints instead of 4, and both frames
resolve at [0.630, +/-0.230, 0.090], matching wheelbase and half-track.

Declaring them <fixed> would also have silenced RViz and would have been
the wrong fix - Gazebo would drag the front wheels instead of rolling
them, corrupting exactly the steering and friction behaviour the twin
exists to reproduce.

Note this obliges Track B: ros2_control validates the URDF against the
hardware plugin, so MittSystem must export these interfaces. The vehicle
has no front-wheel encoders, so it will report a kinematic estimate
(v / wheel_radius), not a measurement, and nothing may treat it as
feedback. Same rule as the shared rear encoder.

Co-Authored-By: Claude Opus 5 (1M context) <noreply@anthropic.com>

File: ros2_ws/src/mitt_description/urdf/mitt_ros2_control.xacro (robot description, xacro)
@@ -50,4 +50,31 @@
         <state_interface name="position"/>
       </joint>
+      <!-- Front road wheels: STATE ONLY, no command interface. These are
+           passive - they free-wheel, nothing drives them.
+           They are listed here purely so joint_state_broadcaster publishes
+           them. Without that, robot_state_publisher cannot compute
+           front_{left,right}_wheel_link, those two frames are ABSENT from TF
+           entirely, and RViz's RobotModel display errors on them.
+           Making them <fixed> would also silence RViz and is the wrong fix:
+           Gazebo would then drag the front wheels instead of rolling them,
+           quietly corrupting the steering and friction behaviour the twin
+           exists to reproduce.
+           HONESTY NOTE, and it matters for Track B. The real vehicle has NO
+           front-wheel encoders. In sim these values are ground truth; on
+           hardware mitt_hardware/MittSystem must still export the interfaces
+           (ros2_control validates the URDF against the plugin and refuses to
+           start on a mismatch), but what it reports will be a KINEMATIC
+           ESTIMATE from vehicle speed, omega = v / wheel_radius, not a
+           measurement. Nothing may consume these as feedback - they exist for
+           visualisation and TF completeness only. Same rule as the shared
+           rear encoder noted above. -->
+      <joint name="front_left_wheel_joint">
+        <state_interface name="position"/>
+        <state_interface name="velocity"/>
+      </joint>
+      <joint name="front_right_wheel_joint">
+        <state_interface name="position"/>
+        <state_interface name="velocity"/>
+      </joint>
     </ros2_control>
     <xacro:if value="${sim}">
