Commit message: Give the vehicle a body mesh, and draw the sensor mounts
Two things.

BODY MESH. Derived from the Fuel "SUV" model by Open Robotics (CC0 -
public domain, chosen over better-looking alternatives carrying
NonCommercial or NoDerivatives terms, same reasoning as the Depot world).
It is a Hummer H2: boxy, upright, flat-roofed, which is the right
silhouette for a Defender-style ride-on.

Three preparation steps, each load-bearing. The source wheel groups are
dropped, because the URDF has its own four wheels that steer and roll and
baked-in ones would sit frozen alongside them. The upstream -90 deg Z
rotation is baked into the vertices rather than left to the URDF origin:
URDF applies <scale> in the mesh frame BEFORE the origin transform, so
with a rotation still pending a non-uniform scale on X would have
stretched the vehicle's width instead of its length. And the mesh is
normalised to a unit bounding box, which is the useful part - <scale> is
then literally the vehicle's size in metres, fed from mitt_dimensions.yaml,
so the shell keeps tracking those numbers when they are finally measured.
No geometric literals, consistent with the rest of the description.

Collision stays a primitive box. Mesh collision would cost physics time
for no gain, and would couple the collision envelope to whatever mesh
happened to be installed.

Gazebo needed GZ_SIM_RESOURCE_PATH to resolve package:// (it rewrites to
model:// and searches only its own path). Without it the vehicle is
invisible while everything else works normally. Set in the launch file so
it cannot be forgotten.

The upstream 753 kB body texture is NOT included: tried both beside the
mesh and under materials/textures/, and it rendered in neither, with no
warning of any kind. Rather than carry an asset that does not draw, the
body is a flat colour stated in both the MTL and the URDF so Gazebo and
RViz agree. It is also more honest - that texture is a photographic
Hummer skin, and grille and badge detail would be misleading on a vehicle
that is not one. Package is 124 kB.

SENSOR DIAGRAMS. Two SVGs answering how the steering and drive sensors
physically attach, since the prose alone left it unclear.

steering-sensing.svg shows the AS5600 on the kingpin axis: magnet bonded
to the rotating shaft, sensor on a chassis-fixed bracket across a
controlled air gap, contactless. It puts the rejected motor-side mounting
next to the adopted one, because the whole point of ADR B is WHERE it
mounts - load-side turns gearbox backlash into measured error instead of
invisible bias.

drive-sensing.svg shows the asymmetry that is easy to miss in prose: both
rear motors paralleled onto one channel, only one instrumented, no
differential. Plus the error chain sitting between that measurement and
actual ground distance - backlash, slip, differential speed in turns -
which is why odometry is fused rather than trusted.

Co-Authored-By: Claude Opus 5 (1M context) <noreply@anthropic.com>

File: ros2_ws/src/mitt_description/urdf/mitt_base.xacro (robot description, xacro)
@@ -39,9 +39,31 @@
   <link name="base_link"/>
   <link name="chassis_link">
+    <!-- Body shell mesh. See meshes/README.md for provenance (Fuel "SUV" by
+         Open Robotics, CC0) and for how it was prepared.
+         NO GEOMETRIC LITERALS HERE EITHER. The mesh is normalised to a unit
+         bounding box - span 1.0 per axis, centred on X/Y, resting on Z=0 - so
+         <scale> below IS the vehicle's size in metres, taken from the same
+         yaml as everything else. The z offset of -body_h/2 lifts the unit box
+         onto the link origin, which is why the mesh occupies EXACTLY the same
+         envelope as the collision box beneath it. Measure the real vehicle,
+         update the yaml, and the shell follows.
+         The mesh is a visual proxy for a Defender-style ride-on, NOT a scan of
+         the donor vehicle. Nothing is dimensioned from it. -->
     <visual>
-      <origin xyz="0 0 0" rpy="0 0 0"/>
-      <geometry><box size="${body_l} ${body_w} ${body_h}"/></geometry>
+      <origin xyz="0 0 ${-body_h/2}" rpy="0 0 0"/>
+      <geometry>
+        <mesh filename="package://mitt_description/meshes/mitt_body.obj"
+              scale="${body_l} ${body_w} ${body_h}"/>
+      </geometry>
+      <!-- Stated explicitly so the colour is deterministic rather than
+           whatever each renderer falls back to. The upstream texture is not
+           used - see meshes/mitt_body.mtl for why. -->
       <material name="mitt_white"/>
     </visual>
+    <!-- Collision stays a PRIMITIVE BOX, deliberately. Mesh collision would
+         cost physics time for no benefit here, and would couple the collision
+         envelope to whatever mesh happens to be installed - so swapping the
+         shell would silently change the vehicle's physics. Keeping the box
+         means the documented dimensions remain the single source of truth. -->
     <collision>
       <origin xyz="0 0 0" rpy="0 0 0"/>

Commit message: Texture the vehicle body, and retract a wrong claim about gz-sim
The body rendered as a flat white shell. meshes/README.md and mitt_body.mtl
both explained why, in these words:

    It was tried both beside the mesh and under materials/textures/ (the gz
    convention), and rendered in neither: gz-sim loads the mesh without any
    warning and simply draws it untextured.

That was wrong, and it was recorded as a fact about the renderer. The
counter-example was running the whole time: the Depot world - the warehouse the
vehicle drives around every session - references ../materials/textures/
WALLS_Albedo.png from Depot.dae by exactly the same relative-path convention,
and draws fully textured.

What actually suppressed the texture was our own description. mitt_base.xacro
put <material name="mitt_white"/> on the mesh visual, and URDF->SDF conversion
turns that into an SDF <material> whose diffuse colour overrides the mesh's own.
There was also a <gazebo><material>Gazebo/White</material> tag, which is Gazebo
CLASSIC script syntax and inert in Harmonic. Two dangling symlinks were still
sitting in install/ pointing at both of the locations the note claimed had
failed - the files had been installed correctly both times and simply painted
over.

The texture is generated rather than taken from upstream. The Fuel model ships a
736 kB photographic Hummer H2 skin, and this mesh only stands in for a
Defender-style 12 V ride-on; painting one real vehicle's bodywork onto a proxy
for a different one asserts something untrue about the platform. scripts/
make_body_texture.py classifies each texel by barycentric interpolation of the
surface point that owns it - height, normal, position - and fills its UV
triangle. 7.5 kB, byte-reproducible.

Per-texel rather than per-face is load-bearing, not gold-plating. This is a
1210-face proxy with no lamp geometry: upstream painted the headlights into its
texture rather than modelling them, so the front is one flat fascia. The first
per-face attempt painted the entire front cream and the entire rear red, which
an offline render caught immediately. Thresholds come from a measured
area-by-height profile, quoted in the script; lamp boxes from the measured
fascia extents.

Wheels get a rim and the sensors get their own colours, because mast, LiDAR,
camera and IMU were all one grey and a wheel was a black puck. Verified in both
renderers, which do NOT agree: Gazebo paints every visual with its own material,
while RViz2 renders all the geometry but applies ONE material per link, taken
from the first visual. So in RViz the rim is a correctly-shaped hub in tyre
black. Left that way deliberately - the fix is a child link per accent, and
decorative frames do not get to pollute a TF tree students read in the Week 5
lab. Documented in both the xacro and the README.

Also fixed a self-inflicted scare while verifying this. A stray colcon build run
from inside src/mitt_description created build/, install/ and log/ IN the
package, and the ament linters then dutifully linted CMake's generated C++ and
cmake files - cpplint failing on CMakeCXXCompilerId.cpp in a package containing
no C++. That produced 143 failures which I was one step away from reporting as a
pre-existing repository problem. It was my own mess. Removed; the workspace is
92 tests, 0 failures.

Co-Authored-By: Claude Opus 5 <noreply@anthropic.com>
Claude-Session: https://claude.ai/code/session_01DRtKXsmjmoJW7KizFXz9KH

File: ros2_ws/src/mitt_description/urdf/mitt_base.xacro (robot description, xacro)
@@ -35,4 +35,9 @@
   <material name="mitt_dark"><color rgba="0.15 0.15 0.15 1.0"/></material>
   <material name="mitt_accent"><color rgba="0.10 0.35 0.65 1.0"/></material>
+  <!-- Wheels/sensors were previously all one of two greys, which made the
+       LiDAR, camera and mast indistinguishable and a wheel a black puck.
+       Orientation legibility is worth real points in every TF and Nav2 lab. -->
+  <material name="mitt_tyre"><color rgba="0.10 0.10 0.11 1.0"/></material>
+  <material name="mitt_rim"><color rgba="0.62 0.63 0.66 1.0"/></material>
   <!-- ==== base_link ======================================================= -->
   <!-- Massless reference frame at the rear axle centre, on the ground. -->
@@ -56,8 +61,9 @@
               scale="${body_l} ${body_w} ${body_h}"/>
       </geometry>
-      <!-- Stated explicitly so the colour is deterministic rather than
-           whatever each renderer falls back to. The upstream texture is not
-           used - see meshes/mitt_body.mtl for why. -->
-      <material name="mitt_white"/>
+      <!-- NO <material> HERE, DELIBERATELY. A material on a mesh visual is
+           converted to an SDF <material> whose diffuse colour OVERRIDES the
+           mesh's own, which is what suppressed the body texture until
+           2026-09-04. Leaving it off lets mitt_body.mtl paint the shell in
+           both Gazebo and RViz. See meshes/README.md for the full correction. -->
     </visual>
     <!-- Collision stays a PRIMITIVE BOX, deliberately. Mesh collision would
@@ -115,5 +121,27 @@
         <origin xyz="0 0 0" rpy="${pi/2} 0 0"/>
         <geometry><cylinder radius="${wheel_r}" length="${wheel_w}"/></geometry>
-        <material name="mitt_dark"/>
+        <material name="mitt_tyre"/>
+      </visual>
+      <!-- Rim: visual only, no collision and no inertia - the tyre cylinder
+           above owns both.
+           It must stand PROUD of the tyre by a real margin. At 1.04x the tyre
+           width the rim face was ~1 mm clear, which is sub-pixel at normal
+           viewing distance and z-fought with the tyre. 1.20x gives 5 mm a
+           side, which reads clearly and still looks like a hub rather than an
+           axle stub.
+           RENDERER DIFFERENCE, verified 2026-09-04. Gazebo paints this its own
+           colour. RViz2's RobotModel display does NOT: it renders the geometry
+           of every visual but applies ONE material per link, taken from the
+           first visual - so in RViz the rim shows as a stepped hub in tyre
+           black. Same applies to the LiDAR cap and camera lens in
+           mitt_sensors.xacro.
+           Left as is deliberately. The fix would be a child link per accent
+           joined by a fixed joint, and that would add half a dozen decorative
+           frames to a TF tree students are asked to read in the Week 5 lab.
+           Cosmetics do not get to pollute the frame graph. -->
+      <visual>
+        <origin xyz="0 0 0" rpy="${pi/2} 0 0"/>
+        <geometry><cylinder radius="${wheel_r*0.55}" length="${wheel_w*1.20}"/></geometry>
+        <material name="mitt_rim"/>
       </visual>
       <collision>
@@ -190,5 +218,9 @@
   <xacro:wheel_gz name="front_left_wheel_link"/>
   <xacro:wheel_gz name="front_right_wheel_link"/>
-  <gazebo reference="chassis_link"><material>Gazebo/White</material></gazebo>
-  <gazebo reference="equipment_plate_link"><material>Gazebo/DarkGrey</material></gazebo>
+  <!-- REMOVED 2026-09-04: <gazebo reference="chassis_link">
+         <material>Gazebo/White</material></gazebo> and its DarkGrey twin.
+       Gazebo/* are Gazebo CLASSIC material-script names with no meaning in
+       Harmonic, so they never did anything - and on the chassis the intent was
+       actively wrong, since the body is now textured from its own MTL. Link
+       colours come from the URDF <material> tags above. -->
 </robot>

File: ros2_ws/src/mitt_description/urdf/mitt_sensors.xacro (robot description, xacro)
@@ -20,4 +20,12 @@
   <xacro:property name="body_hh"     value="${ds['chassis_height']}"/>
   <material name="mast_grey"><color rgba="0.35 0.35 0.35 1.0"/></material>
+  <!-- Distinct per sensor. These were all mast_grey, which made the LiDAR,
+       camera and IMU indistinguishable from the pole they hang off - a
+       genuine nuisance when a lab asks "where is base_link -> laser_link?" -->
+  <material name="lidar_body"><color rgba="0.12 0.13 0.15 1.0"/></material>
+  <material name="lidar_cap"><color rgba="0.85 0.62 0.10 1.0"/></material>
+  <material name="camera_body"><color rgba="0.16 0.17 0.19 1.0"/></material>
+  <material name="camera_lens"><color rgba="0.20 0.45 0.70 1.0"/></material>
+  <material name="imu_body"><color rgba="0.20 0.55 0.30 1.0"/></material>
   <!-- ==== Mast ============================================================ -->
   <xacro:property name="mast_r" value="0.015"/>
@@ -47,5 +55,10 @@
     <visual>
       <geometry><cylinder radius="0.038" length="0.041"/></geometry>
-      <material name="mast_grey"/>
+      <material name="lidar_body"/>
+    </visual>
+    <visual>
+      <origin xyz="0 0 0.0215" rpy="0 0 0"/>
+      <geometry><cylinder radius="0.0345" length="0.006"/></geometry>
+      <material name="lidar_cap"/>
     </visual>
     <collision>
@@ -96,5 +109,10 @@
     <visual>
       <geometry><box size="0.03 0.09 0.025"/></geometry>
-      <material name="mast_grey"/>
+      <material name="camera_body"/>
+    </visual>
+    <visual>
+      <origin xyz="0.016 0 0" rpy="0 ${pi/2} 0"/>
+      <geometry><cylinder radius="0.009" length="0.003"/></geometry>
+      <material name="camera_lens"/>
     </visual>
     <xacro:inertial_box mass="0.08" x="0.03" y="0.09" z="0.025">
@@ -138,5 +156,5 @@
     <visual>
       <geometry><box size="0.02 0.02 0.006"/></geometry>
-      <material name="mast_grey"/>
+      <material name="imu_body"/>
     </visual>
     <xacro:inertial_box mass="0.01" x="0.02" y="0.02" z="0.006">
